File: PCB-house/PCB-house.kicad_pcb (KiCad board)
At the start: 2 copper layers, 100 x 80 mm, 45 parts, among them J1 DIN-5_180degree, J2 DIN-5_180degree, J3 DIN-5_180degree, J4 DIN-5_180degree, J5 DIN-5_180degree, Q1 BC547, Q2 BC547, Q3 BC547, Q4 BC547, U1 6N138, U2 L7805

Commit message: Getting there
Parts:
- removed +5v1: Conn_01x01, Connector_Wire:SolderWire-1.5sqmm_1x01_D1.7mm_OD3.9mm
- removed the Q2 at (58.4, 55.9)
- removed the R10 at (48.3, 41.9)
- removed the R11 at (52.1, 52.1)
- removed the R12 at (43.2, 52.1)
- removed the R9 at (58.4, 41.9)
- added -12v1: Conn_01x01, Connector_Wire:SolderWire-1.5sqmm_1x01_D1.7mm_OD3.9mm, F.Cu at (148.6, 39.7)
- added C5: 10µ 25v, Capacitor_THT:CP_Radial_D5.0mm_P2.00mm, F.Cu at (147.7, 50.6)
- added D2: 1N4148, Diode_THT:D_DO-35_SOD27_P10.16mm_Horizontal, F.Cu at (133.6, 42.0)
- added D3: 1N4148, Diode_THT:D_DO-35_SOD27_P10.16mm_Horizontal, F.Cu at (133.6, 45.6)
- added D4: 1N4148, Diode_THT:D_DO-35_SOD27_P10.16mm_Horizontal, F.Cu at (133.6, 38.5)
- added Q4: BC557, Package_TO_SOT_THT:TO-92_Inline, F.Cu at (147.3, 57.1)
- added R17: 82R, PCM_Resistor_THT_AKL:R_Axial_DIN0207_L6.3mm_D2.5mm_P10.16mm_Horizontal, F.Cu at (133.6, 49.4)
- added R18: 2k2, PCM_Resistor_THT_AKL:R_Axial_DIN0207_L6.3mm_D2.5mm_P10.16mm_Horizontal, F.Cu at (133.6, 53.4)
- added R19: 2k7, PCM_Resistor_THT_AKL:R_Axial_DIN0207_L6.3mm_D2.5mm_P10.16mm_Horizontal, F.Cu at (133.6, 57.5)
- added R20: 1k8, PCM_Resistor_THT_AKL:R_Axial_DIN0207_L6.3mm_D2.5mm_P10.16mm_Horizontal, F.Cu at (133.6, 61.5)
- moved Q2 99.4 mm to (148.6, 113.0)
- moved Q3 97.3 mm to (156.2, 113.0)
- moved R10 97.0 mm to (148.6, 100.3)
- moved R12 97.0 mm to (152.4, 100.3)
- moved R15 97.0 mm to (144.8, 110.5)
- moved R16 97.0 mm to (141.0, 110.5)
- moved R9 96.0 mm to (160.0, 100.3)
- moved R11 96.0 mm to (156.2, 110.5)
- moved J5 93.4 mm to (111.6, 127.0)
- moved R4 93.0 mm to (163.8, 110.5)
- moved R3 93.0 mm to (182.9, 100.3)
- moved R1 93.0 mm to (167.6, 100.3)
- moved R2 93.0 mm to (175.3, 100.3)
- moved R5 93.0 mm to (171.4, 110.5)
- moved R6 93.0 mm to (179.1, 110.5)
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- renumbered +12v to +12v1, C2 to C1, C3 to C2, C4 to C3, C1 to C4, H4 to H2, H2 to H3, H3 to H4, Q3 to Q2, Q4 to Q3, R4 to R1, R17 to R10, R19 to R11, R18 to R12, R14 to R13, R13 to R14, R6 to R2, R8 to R3, R3 to R4, R7 to R6, R1 to R7, R2 to R8, R20 to R9, U2 to U1, U1 to U2
Routing:
- net +5V: track 189.8 -> 17.1 mm
- net Net-(J5-Pad5): track 122.3 -> 0.00 mm, vias 2 -> 0
- net Net-(J5-Pad4): track 69.9 -> 0.00 mm
- net Net-(U2-VO2): track 62.3 -> 0.00 mm
- net Net-(Q4-C): track 52.1 -> 0.00 mm, vias 2 -> 0
- net Net-(J4-Pad4): track 27.1 -> 0.00 mm
- net Net-(Q1-C): track 43.2 -> 17.3 mm
- net Net-(D1-K): track 25.4 -> 0.00 mm
- net Net-(Q2-B) (its old number): track 24.4 -> 0.00 mm
- net Net-(+12v1-Pin_1): track 22.9 -> 0.00 mm
- net Net-(Q2-C): track 19.4 -> 0.00 mm
- net Net-(U2-C2): track 18.4 -> 0.00 mm
- net Net-(J3-Pad4): track 32.0 -> 16.1 mm
- net Net-(Q2-B): track 14.0 -> 0.00 mm
- net Net-(J4-PadMH1): track 10.0 -> 0.00 mm
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- removed copper zone on B.Cu, net GND
- removed copper zone on F.Cu, net GND
Other:
- board outline removed
