File: PCB-house/PCB-house.kicad_sch (KiCad schematic)
At the start: 45 parts, among them J1 DIN-5_180degree, J2 DIN-5_180degree, J3 DIN-5_180degree, J4 DIN-5_180degree, J5 DIN-5_180degree, Q1 BC547, Q2 BC547, Q3 BC547, Q4 BC547, U1 6N138, U2 L7805

Commit message: Getting there
Parts:
- removed +5v1: Conn_01x01, Connector_Wire:SolderWire-1.5sqmm_1x01_D1.7mm_OD3.9mm, symbol Connector_Generic:Conn_01x01
- removed Q2: BC547, PCM_Package_TO_SOT_THT_AKL:TO-92_Inline_Wide_CBE, symbol PCM_Transistor_BJT_AKL:BC547
- removed R10, R12: 1k5, PCM_Resistor_THT_AKL:R_Axial_DIN0207_L6.3mm_D2.5mm_P10.16mm_Horizontal, symbol Device:R
- removed R11: 5k6, PCM_Resistor_THT_AKL:R_Axial_DIN0207_L6.3mm_D2.5mm_P10.16mm_Horizontal, symbol Device:R
- removed R9: 1k, PCM_Resistor_THT_AKL:R_Axial_DIN0207_L6.3mm_D2.5mm_P10.16mm_Horizontal, symbol Device:R
- added -12v1: Conn_01x01, Connector_Wire:SolderWire-1.5sqmm_1x01_D1.7mm_OD3.9mm, symbol Connector_Generic:Conn_01x01
- added C5: 10µ 25v, Capacitor_THT:CP_Radial_D5.0mm_P2.00mm, symbol Device:C_Polarized
- added D2, D3, D4: 1N4148, Diode_THT:D_DO-35_SOD27_P10.16mm_Horizontal, symbol PCM_Diode_AKL:1N4148
- added Q4: BC557, Package_TO_SOT_THT:TO-92_Inline, symbol Transistor_BJT:BC557
- added R17: 82R, PCM_Resistor_THT_AKL:R_Axial_DIN0207_L6.3mm_D2.5mm_P10.16mm_Horizontal, symbol Device:R
- added R18: 2k2, PCM_Resistor_THT_AKL:R_Axial_DIN0207_L6.3mm_D2.5mm_P10.16mm_Horizontal, symbol Device:R
- added R19: 2k7, PCM_Resistor_THT_AKL:R_Axial_DIN0207_L6.3mm_D2.5mm_P10.16mm_Horizontal, symbol Device:R
- added R20: 1k8, PCM_Resistor_THT_AKL:R_Axial_DIN0207_L6.3mm_D2.5mm_P10.16mm_Horizontal, symbol Device:R
- renumbered C2 to C1, C3 to C2, C4 to C3, C1 to C4, H4 to H2, H2 to H3, H3 to H4, Q3 to Q2, Q4 to Q3, R4 to R1, R17 to R10, R19 to R11, R18 to R12, R14 to R13, R13 to R14, R6 to R2, R8 to R3, R3 to R4, R7 to R6, R1 to R7, R2 to R8, R20 to R9, U2 to U1, U1 to U2
Connections:
- net +5V: now also R17.1, R18.1
- net GND: now also C5.1, D4.1 (K)
- net at RXD1.1 (Pin_1): now also Q4.1 (C), R20.1
- net at R15.2, U2.6 (VO2): now also R19.2
- net at R7.2, TXD1.1 (Pin_1): now also D2.2 (A)
- new net: C5.2, D2.1 (K), D3.2 (A), D4.2 (A), R20.2
- new net: -12v1.1 (Pin_1), D3.1 (K)
- new net: Q4.2 (B), R18.2, R19.1
- new net: Q4.3 (E), R17.2
Other:
- moved on the sheet: C4, D1, GND1, H1, H2, H3, H4, J1, J2, J3, J4, J5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
