File: PCB-House/PCB-House.kicad_pcb (KiCad board)
At the start: 2 copper layers, 100 x 80 mm, 48 parts, among them J1 DIN-5_180degree, J2 DIN-5_180degree, J3 DIN-5_180degree, J4 DIN-5_180degree, J5 DIN-5_180degree, Q1 BC547, Q2 BC557, Q3 BC547, Q4 BC547, U1 L7805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

Commit message: PCB-house done
Parts:
- added D3: 1N4148, Diode_THT:D_DO-35_SOD27_P10.16mm_Horizontal, F.Cu at (61.0, 38.7)
- added R21: 1k5, PCM_Resistor_THT_AKL:R_Axial_DIN0207_L6.3mm_D2.5mm_P10.16mm_Horizontal, F.Cu at (73.7, 38.7)
- moved R13 19.3 mm to (65.4, 66.0), turned to 180 degrees
- moved Q4 5.09 mm to (77.5, 61.0), turned to 90 degrees
Connections:
- R16 pad 2: Net-(U2-VO2) -> Net-(D3-A)
- R18 pad 2: Net-(U2-VO2) -> Net-(D3-K)
- U2 pad 6: Net-(U2-VO2) -> Net-(D3-K)
Routing:
- net Net-(J5-Pad5): track 103.2 -> 40.3 mm, vias 2 -> 0
- net Net-(D3-K): track 0.00 -> 37.5 mm
- net Net-(U2-VO2): track 34.3 -> 0.00 mm
- net Net-(Q4-C): track 5.09 -> 15.7 mm
- net +5V: track 169.0 -> 176.6 mm
- net Net-(D3-A): track 0.00 -> 3.17 mm
- net GND: vias 0 -> 2
