File: PCB-House/PCB-House.kicad_sch (KiCad schematic)
At the start: 48 parts, among them J1 DIN-5_180degree, J2 DIN-5_180degree, J3 DIN-5_180degree, J4 DIN-5_180degree, J5 DIN-5_180degree, Q1 BC547, Q2 BC557, Q3 BC547, Q4 BC547, U1 L7805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

Commit message: PCB-house done
Parts:
- added D3: 1N4148, Diode_THT:D_DO-35_SOD27_P10.16mm_Horizontal, symbol PCM_Diode_AKL:1N4148
- added R21: 1k5, PCM_Resistor_THT_AKL:R_Axial_DIN0207_L6.3mm_D2.5mm_P10.16mm_Horizontal, symbol Device:R
- Q2: footprint Package_TO_SOT_THT:TO-92_Inline -> Package_TO_SOT_THT:TO-92_Inline_Wide
Connections:
- net +5V: now also R21.1
- net at R18.2, U2.6 (VO2): now also D3.1 (K), R21.2; no longer R16.2
- new net: D3.2 (A), R16.2
Other:
- moved on the sheet: GND1, Q2, R10, R12, R16
